File: tigard.kicad_pcb (KiCad board)
At the start: 4 copper layers, 46 x 46 mm, 92 parts, among them J1 USB_C_Receptacle_USB2.0, J2 JTAG, J3 UART, J4 SPI, J5 CORTEX, J6 LA, J7 I2C, Q1 BSH103, SW1 TARGET, SW2 MODE, U1 AP7365-18, U2 AP7365-33, U3 FT2232HQ, U4 93LC46BT-I/OT, U5 SN74LVC8T245, U6 SN74LVC8T245, Y1 12MHz

Commit message: switch to kicad 10
Connections:
- net /~ENABLE renamed /~{ENABLE}
- net /~UART_CTS renamed /~{UART_CTS}
- net /~UART_DCD renamed /~{UART_DCD}
- net /~UART_DSR renamed /~{UART_DSR}
- net /~UART_DTR renamed /~{UART_DTR}
- net /~UART_RTS renamed /~{UART_RTS}
Routing:
- added copper zone on In2.Cu, net +3V3
- added copper zone on In1.Cu, net GND
- removed copper zone on PWR, net +3V3
- removed copper zone on GND, net GND
Other:
- net class Default removed

Commit message: fix I2C reading
Parts:
- removed LOGO2: Logo_SH, tigard:Securing_Hardware_Logo
- moved J7 47.4 mm to (65.8, 33.1), turned to 180 degrees
- moved TP1 38.3 mm to (39.9, 72.0)
- moved J3 7.04 mm to (39.3, 33.7)
- moved R16 4.63 mm to (66.2, 42.5)
- moved JP2 3.85 mm to (67.6, 40.8)
- moved SW2 0.61 mm to (59.0, 40.8)
Connections:
- J1 pad A8: (no net) -> unconnected-(J1-SBU1-PadA8)
- J1 pad B8: (no net) -> unconnected-(J1-SBU2-PadB8)
- J2 pad 4: /COPI -> /DO
- J2 pad 5: /CIPO -> /TDO
- J4 pad 3: /CIPO -> /DI
- J4 pad 8: /COPI -> /DO
- J5 pad 6: /CIPO -> /TDO
- J5 pad 7: (no net) -> unconnected-(J5-Pin_7-Pad7)
- J5 pad 8: /COPI -> /DO
- J6 pad 11: (no net) -> unconnected-(J6-Pin_11-Pad11)
- J6 pad 12: (no net) -> unconnected-(J6-Pin_12-Pad12)
- J6 pad 13: (no net) -> unconnected-(J6-Pin_13-Pad13)
- J6 pad 14: (no net) -> unconnected-(J6-Pin_14-Pad14)
- J6 pad 2: /COPI -> /DO
- J7 pad 3: /COPI -> /DIO
- JP2 pad 1: /COPI -> /DO
- JP2 pad 2: /SWDIO -> /DIO
- R16 pad 1: /SWDIO -> /DIO
- R16 pad 2: /COPI -> /DO
- RN3 pad 7: /COPI -> /DO
- RN6 pad 3: (no net) -> unconnected-(RN6-R3.1-Pad3)
- RN6 pad 4: (no net) -> unconnected-(RN6-R4.1-Pad4)
- SW1 pad 1: (no net) -> unconnected-(SW1-Pad1)
- SW1 pad 2: (no net) -> unconnected-(SW1-Pad2)
- SW1 pad 3: (no net) -> unconnected-(SW1-Pad3)
- SW1 pad 4: (no net) -> unconnected-(SW1-Pad4)
- SW1 pad 5: (no net) -> unconnected-(SW1-Pad5)
- SW2 pad 3: /SWDIO -> /DIO
- SW2 pad 4: /CIPO -> /TDO
- SW2 pad 6: /SWDIO -> /DIO
- U1 pad 4: (no net) -> unconnected-(U1-NC-Pad4)
- U2 pad 4: (no net) -> unconnected-(U2-NC-Pad4)
- U3 pad 24: (no net) -> unconnected-(U3-ADBUS7-Pad24)
- U3 pad 26: (no net) -> unconnected-(U3-ACBUS0-Pad26)
- U3 pad 27: (no net) -> unconnected-(U3-ACBUS1-Pad27)
- U3 pad 28: (no net) -> unconnected-(U3-ACBUS2-Pad28)
- U3 pad 32: (no net) -> unconnected-(U3-ACBUS5-Pad32)
- U3 pad 33: (no net) -> unconnected-(U3-ACBUS6-Pad33)
- U3 pad 34: (no net) -> unconnected-(U3-ACBUS7-Pad34)
- U3 pad 36: (no net) -> unconnected-(U3-~{SUSPEND}-Pad36)
- U3 pad 48: (no net) -> unconnected-(U3-BCBUS0-Pad48)
- U3 pad 52: (no net) -> unconnected-(U3-BCBUS1-Pad52)
- U3 pad 53: (no net) -> unconnected-(U3-BCBUS2-Pad53)
- U3 pad 54: (no net) -> unconnected-(U3-BCBUS3-Pad54)
- U3 pad 55: (no net) -> unconnected-(U3-BCBUS4-Pad55)
- U3 pad 57: (no net) -> unconnected-(U3-BCBUS5-Pad57)
- U3 pad 58: (no net) -> unconnected-(U3-BCBUS6-Pad58)
- U3 pad 59: (no net) -> unconnected-(U3-BCBUS7-Pad59)
Routing:
- net /COPI: track 104.5 -> 0.00 mm, vias 3 -> 0
- net /DO: track 0.00 -> 73.1 mm, vias 0 -> 3
- net /CIPO: track 64.5 -> 0.00 mm, vias 1 -> 0
- net /TDO: track 0.00 -> 43.3 mm, vias 0 -> 1
- net /CLK: track 87.3 -> 75.0 mm
- net /DIO: track 0.00 -> 11.6 mm
- net /SWDIO: track 10.1 -> 0.00 mm
- net /UART_TX: track 63.0 -> 70.5 mm
- net /~{UART_DCD}: track 30.9 -> 24.3 mm
- net /ICE_CDONE: track 74.9 -> 81.2 mm
- net /~{UART_RTS}: track 36.3 -> 41.5 mm
- net /DI: track 56.2 -> 61.0 mm, vias 3 -> 4
- net /~{UART_DSR}: track 28.2 -> 23.8 mm
- net /~{UART_CTS}: track 24.0 -> 26.2 mm
- net /~{UART_DTR}: track 37.6 -> 35.5 mm
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Other:
- board text added: "v1.1.1"
- board text added: "© Franklin Harding 2020 (upd by GrKa) CC-BY-SA 4.0"
- board text removed: "securinghw.com"
- board text removed: "v1.1"
- board text removed: "© Franklin Harding 2020 CC-BY-SA 4.0"
