File: tigard.kicad_sch (KiCad schematic)
At the start: 91 parts, among them J1 USB_C_Receptacle_USB2.0, J2 JTAG, J3 UART, J4 SPI, J5 CORTEX, J6 LA, J7 I2C, Q1 BSH103, SW1 TARGET, SW2 MODE, U1 AP7365-18, U2 AP7365-33, U3 FT2232HQ, U4 93LC46BT-I/OT, U5 SN74LVC8T245, U6 SN74LVC8T245, Y1 12MHz

Commit message: fix I2C reading
Connections:
- net DI: now also J4.3 (Pin_3)
- net CIPO renamed TDO
- net TDO: no longer J4.3 (Pin_3)
- net COPI renamed DO
- net DO: no longer J7.3 (Pin_3)
- net SWDIO renamed DIO
- net DIO: now also J7.3 (Pin_3)
Changed lines of the file:
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@@
 	(wire
 		(pts
+			(xy 163.83 85.09) (xy 170.18 85.09)
+		)
+		(stroke
+			(width 0)
+			(type default)
+		)
+	)
+	(wire
+		(pts
 			(xy 196.85 113.03) (xy 196.85 114.3)
 		)
@@
 	(wire
 		(pts
+			(xy 205.74 91.44) (xy 215.9 91.44)
+		)
+		(stroke
+			(width 0)
+			(type default)
+		)
+	)
+	(wire
+		(pts
 			(xy 217.17 190.5) (xy 217.17 193.04)
 		)
@@
 	(wire
 		(pts
-			(xy 204.47 90.17) (xy 218.44 90.17)
-		)
-		(stroke
-			(width 0)
-			(type default)
-		)
-	)
-	(wire
-		(pts
 			(xy 228.6 58.42) (xy 228.6 67.31)
 		)
@@
 	(wire
 		(pts
-			(xy 158.75 85.09) (xy 170.18 85.09)
-		)
-		(stroke
-			(width 0)
-			(type default)
-		)
-	)
-	(wire
-		(pts
 			(xy 161.29 22.86) (xy 161.29 24.13)
 		)
@@
 		)
 	)
-	(label "SWDIO"
+	(label "DIO"
 		(at 158.75 90.17 0)
 		(effects
@@
 		)
 	)
-	(label "xPB4"
-		(at 236.22 82.55 0)
+	(label "SWDIO"
+		(at 163.83 99.06 0)
 		(effects
 			(font
@@
 		)
 	)
-	(label "TMS"
-		(at 162.56 93.98 0)
+	(label "xPB4"
+		(at 236.22 82.55 0)
 		(effects
 			(font
@@
 		)
 	)
+	(label "CS"
+		(at 158.75 93.98 0)
+		(effects
+			(font
+				(size 1.27 1.27)
+			)
+			(justify left bottom)
+		)
+	)
+	(label "CLK"
+		(at 205.74 91.44 0)
+		(effects
+			(font
+				(size 1.27 1.27)
+			)
+			(justify left bottom)
+		)
+	)
 	(label "xPB7"
 		(at 194.31 187.96 180)
@@
 		)
 	)
-	(label "COPI"
-		(at 140.97 95.25 180)
+	(label "TMS"
+		(at 163.83 93.98 0)
 		(effects
 			(font
 				(size 1.27 1.27)
 			)
-			(justify right bottom)
+			(justify left bottom)
 		)
 	)
@@
 		)
 	)
+	(label "TCK"
+		(at 215.9 91.44 180)
+		(effects
+			(font
+				(size 1.27 1.27)
+			)
+			(justify right bottom)
+		)
+	)
 	(label "UART_RX"
 		(at 204.47 187.96 180)
@@
 	)
 	(label "TDO"
-		(at 165.1 85.09 0)
+		(at 163.83 85.09 0)
 		(effects
 			(font
@@
 		)
 	)
-	(label "CS"
-		(at 158.75 93.98 0)
-		(effects
-			(font
-				(size 1.27 1.27)
-			)
-			(justify left bottom)
-		)
-	)
-	(label "TDI"
-		(at 132.08 95.25 0)
-		(effects
-			(font
-				(size 1.27 1.27)
-			)
-			(justify left bottom)
-		)
-	)
 	(label "EEDATA"
 		(at 30.48 186.69 0)
@@
 		)
 	)
-	(label "CIPO"
+	(label "DI"
 		(at 234.95 55.88 0)
 		(effects
@@
 		)
 	)
-	(label "COPI"
+	(label "DIO"
 		(at 294.64 93.98 180)
 		(effects
@@
 		)
 	)
-	(label "CIPO"
-		(at 158.75 85.09 0)
-		(effects
-			(font
-				(size 1.27 1.27)
-			)
-			(justify left bottom)
-		)
-	)
 	(label "BD0"
 		(at 152.4 140.97 0)
@@
 		)
 	)
-	(label "COPI"
+	(label "DO"
 		(at 261.62 60.96 180)
 		(effects
@@
 		)
 	)
+	(label "TDI"
+		(at 135.89 95.25 180)
+		(effects
+			(font
+				(size 1.27 1.27)
+			)
+			(justify right bottom)
+		)
+	)
 	(label "EECS"
 		(at 48.26 254 0)
@@
 		)
 	)
-	(label "SWDIO"
+	(label "DIO"
 		(at 158.75 99.06 0)
 		(effects
@@
 		)
 	)
-	(label "CLK"
-		(at 204.47 90.17 0)
-		(effects
-			(font
-				(size 1.27 1.27)
-			)
-			(justify left bottom)
-		)
-	)
-	(label "TCK"
-		(at 218.44 90.17 180)
-		(effects
-			(font
-				(size 1.27 1.27)
-			)
-			(justify right bottom)
-		)
-	)
